File: pcb_v2/upsy-desky.kicad_pcb (KiCad board)
At the start: 2 copper layers, 40.9 x 58 mm, 62 parts, among them J1 RJ45, J2 RJ45, J3 USB_C_ReceptacleUSB2.0, J4 Conn_01x03_Socket, J5 Screw_Terminal_01x03, J6 Conn_01x03_Pin, Q3 2N7002, Q4 2N7002, Q5 2N7002, Q6 2N7002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

Commit message: Updated BOM for PCBWay
Parts:
- turned R5 to 180 degrees
Connections:
- R5 pad 1: +3V3 -> /EN
- R5 pad 2: /EN -> +3V3
Routing:
- net VBUS: track 60.0 -> 57.5 mm
